File: MCS-48_EVB.kicad_pcb (KiCad board)
At the start: 2 copper layers, 37 parts, among them CON1 BARREL_JACK, P1 CONN_01X06, P10 CONN_01X08, P11 CONN_01X06, P2 CONN_01X06, P3 CONN_01X08, P4 CONN_01X08, P5 CONN_01X03, P6 CONN_01X03, P7 CONN_01X02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

Commit message: Corrected gerber files
Other:
- board outline added: 141 x 103.7 mm
Changed lines of the file:
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@@
     (area 26.417599 48.154266 170.438134 155.401333)
     (thickness 1.6)
-    (drawings 9)
+    (drawings 14)
     (tracks 1449)
     (zones 0)
@@
     )
   )
+  (gr_line (start 26.4414 152.6032) (end 26.4922 152.6032) (angle 90) (layer Edge.Cuts) (width 0.15))
+  (gr_line (start 26.4414 48.8696) (end 26.4414 152.6032) (angle 90) (layer Edge.Cuts) (width 0.15))
+  (gr_line (start 167.4622 48.8696) (end 26.4668 48.8696) (angle 90) (layer Edge.Cuts) (width 0.15))
+  (gr_line (start 167.4622 152.6032) (end 167.4622 48.8696) (angle 90) (layer Edge.Cuts) (width 0.15))
+  (gr_line (start 26.4668 152.6032) (end 167.4622 152.6032) (angle 90) (layer Edge.Cuts) (width 0.15))
   (gr_line (start 26.5176 152.5524) (end 26.5176 152.527) (angle 90) (layer Margin) (width 0.2))
   (gr_line (start 31.8008 152.5524) (end 26.5176 152.5524) (angle 90) (layer Margin) (width 0.2))
